Commit message: coba navigation pakai code

File: chapter4_tutorials/robot1_description/urdf/robot1.urdf (robot description, URDF)
Before this commit: robot Robot1, 5 links, 4 joints
Links:
- added link arm_1, mass 1; collision box size=0.05 .05 0.5; visual box size=0.05 .05 0.5
- added link arm_2, mass 1; collision box size=0.05 .05 0.5; visual box size=0.05 0.05 0.5
- added link arm_base, mass 1; collision box size=0.1 .1 .1; visual box size=0.1 .1 .1
- added link left_gripper, mass 1; collision box size=0.1 .1 .1; visual mesh filename=package://pr2_description/meshes/gripper_v0/l_finger.dae
- added link left_tip, mass 1; collision box size=0.1 .1 .1; visual mesh filename=package://pr2_description/meshes/gripper_v0/l_finger_tip.dae
- added link right_gripper, mass 1; collision box size=0.1 .1 .1; visual mesh filename=package://pr2_description/meshes/gripper_v0/l_finger.dae
- added link right_tip, mass 1; collision box size=0.1 .1 .1; visual mesh filename=package://pr2_description/meshes/gripper_v0/l_finger_tip.dae
- link base_link: mass None -> 100; geometry collision box size=0.2 .3 0.1; visual box size=0.2 .3 .1
- link wheel_1: mass None -> 10; geometry collision cylinder length=0.05 radius=0.05; visual cylinder length=0.05 radius=0.05
- link wheel_2: mass None -> 10; geometry collision cylinder length=0.05 radius=0.05; visual cylinder length=0.05 radius=0.05
- link wheel_3: mass None -> 10; geometry collision cylinder length=0.05 radius=0.05; visual cylinder length=0.05 radius=0.05
- link wheel_4: mass None -> 10; geometry collision cylinder length=0.05 radius=0.05; visual cylinder length=0.05 radius=0.05
Joints:
- added joint arm_1_to_arm_base: type revolute, parent arm_base, child arm_1, origin xyz=0 0 0.15, axis 1 0 0, limit lower=-1.0 upper=1.0 effort=1000.0 velocity=0.5
- added joint arm_2_to_arm_1: type revolute, parent arm_1, child arm_2, origin xyz=0.0 0 0.45, axis 1 0 0, limit lower=-2.5 upper=2.5 effort=1000.0 velocity=0.5
- added joint base_to_arm_base: type continuous, parent base_link, child arm_base, origin xyz=0 0 0, axis 0 0 1
- added joint left_gripper_joint: type revolute, parent arm_2, child left_gripper, origin xyz=0.06 0 0.4 rpy=0 -1.57 0, axis 0 0 1, limit lower=0.0 upper=0.548 effort=1000.0 velocity=0.5
- added joint left_tip_joint: type fixed, parent left_gripper, child left_tip
- added joint right_gripper_joint: type revolute, parent arm_2, child right_gripper, origin xyz=0.06 0 0.4 rpy=0 -1.57 0, axis 0 0 -1, limit lower=0.0 upper=0.548 effort=1000.0 velocity=0.5
- added joint right_tip_joint: type fixed, parent right_gripper, child right_tip
